File: 1.1 - Sensor de temperatura/Sensor de temperatura.brd (EAGLE design)
At the start: 155.4 x 59.7 mm, 11 parts, among them U1 ARDUINO-UNO-R3-SHIELD

Commit message: Refactoring the code and some files
Parts:
- moved R4 132.1 mm to (215.1, 35.6)
- moved RR5_TERRA 115.0 mm to (203.2, 32.9)
- moved RR6_TERRA 95.2 mm to (189.3, 30.3)
- moved D3 2.54 mm to (149.8, 36.2)
- moved R3 2.54 mm to (150.9, 29.2)
Connections:
- net U1_GND: no longer R3.1
Other:
- board size 155.4 x 59.7 mm -> 221.4 x 59.7 mm
